File: KiCAD/GateEX/GateEX.kicad_pcb (KiCad board)
At the start: 2 copper layers, 94 x 71.1 mm, 28 parts, among them J1 SYNC_THRU, J2 SYNC_IN, J3 GATE_OUT_1, J4 GATE_OUT_2, J5 PWR_IN, J6 TP_GND, SW1 SEQUENCE1, SW2 SEQUENCE2, U1 Arduino_Pro_Mini, U2 Arduino_Pro_Mini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

Commit message: Comletion
Routing:
- net GND: track 0.00 -> 331.4 mm
- net +5V: track 0.00 -> 113.6 mm, vias 0 -> 4
- net Net-(D1-Pad1): track 0.00 -> 56.9 mm, vias 0 -> 2
- net Net-(J3-Pad1): track 0.00 -> 49.3 mm, vias 0 -> 2
- net Net-(J4-Pad1): track 0.00 -> 47.8 mm, vias 0 -> 2
- net Net-(J1-Pad1): track 0.00 -> 20.3 mm
- net /S08: track 0.00 -> 18.8 mm
- net /S18: track 0.00 -> 18.8 mm
- net Net-(C1-Pad1): track 0.00 -> 18.8 mm
- net Net-(RV2-Pad2): track 0.00 -> 7.69 mm
- net Net-(RV1-Pad2): track 0.00 -> 7.64 mm
- net Net-(R3-Pad2): track 0.00 -> 2.54 mm
- net Net-(R2-Pad2): track 0.00 -> 2.54 mm
- net /S17: track 0.00 -> 2.54 mm
- net /S16: track 0.00 -> 2.54 mm
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